Commit message: isaac sim fix with gripper working version

File: src/ros2_robotiq_gripper/robotiq_description/urdf/2f_140.ros2_control.xacro (robot description, xacro)
@@ -18,84 +18,4 @@
       gripper_max_force:=125.0
       gripper_closed_position:=0.695">
-    <ros2_control name="${name}" type="system">
-      <hardware>
-        <!-- EXACTLY ONE plugin should be selected -->
-        <xacro:if value="${sim_isaac}">
-          <plugin>topic_based_ros2_control/TopicBasedSystem</plugin>
-          <param name="joint_commands_topic">${isaac_joint_commands}</param>
-          <param name="joint_states_topic">${isaac_joint_states}</param>
-        </xacro:if>
-        <xacro:if value="${(not sim_isaac) and sim_ignition}">
-          <plugin>ign_ros2_control/IgnitionSystem</plugin>
-        </xacro:if>
-        <xacro:if value="${(not sim_isaac) and (not sim_ignition) and use_fake_hardware}">
-          <plugin>mock_components/GenericSystem</plugin>
-          <param name="mock_sensor_commands">${mock_sensor_commands}</param>
-          <param name="state_following_offset">0.0</param>
-        </xacro:if>
-        <xacro:if value="${(not sim_isaac) and (not sim_ignition) and (not use_fake_hardware)}">
-          <plugin>robotiq_driver/RobotiqGripperHardwareInterface</plugin>
-          <param name="gripper_closed_position">${gripper_closed_position}</param>
-          <param name="COM_port">${com_port}</param>
-          <param name="gripper_speed_multiplier">${gripper_speed_multiplier}</param>
-          <param name="gripper_force_multiplier">${gripper_force_multiplier}</param>
-          <param name="gripper_max_speed">${gripper_max_speed}</param>
-          <param name="gripper_max_force">${gripper_max_force}</param>
-        </xacro:if>
-      </hardware>
-      <!-- Joint interfaces -->
-      <joint name="${prefix}finger_joint">
-        <command_interface name="position"/>
-        <state_interface name="position">
-          <param name="initial_value">${gripper_closed_position}</param>
-        </state_interface>
-        <state_interface name="velocity"/>
-      </joint>
-      <!-- When simulating we include the rest of the mimic joints -->
-      <xacro:if value="${use_fake_hardware or sim_isaac or sim_ignition}">
-        <joint name="${prefix}left_inner_knuckle_joint">
-          <param name="mimic">${prefix}finger_joint</param>
-          <param name="multiplier">-1</param>
-          <command_interface name="position"/>
-          <state_interface name="position"/>
-          <state_interface name="velocity"/>
-        </joint>
-        <joint name="${prefix}left_inner_finger_joint">
-          <param name="mimic">${prefix}finger_joint</param>
-          <param name="multiplier">1</param>
-          <command_interface name="position"/>
-          <state_interface name="position"/>
-          <state_interface name="velocity"/>
-        </joint>
-        <joint name="${prefix}right_outer_knuckle_joint">
-          <param name="mimic">${prefix}finger_joint</param>
-          <param name="multiplier">-1</param>
-          <command_interface name="position"/>
-          <state_interface name="position"/>
-          <state_interface name="velocity"/>
-        </joint>
-        <joint name="${prefix}right_inner_knuckle_joint">
-          <param name="mimic">${prefix}finger_joint</param>
-          <param name="multiplier">-1</param>
-          <command_interface name="position"/>
-          <state_interface name="position"/>
-          <state_interface name="velocity"/>
-        </joint>
-        <joint name="${prefix}right_inner_finger_joint">
-          <param name="mimic">${prefix}finger_joint</param>
-          <param name="multiplier">1</param>
-          <command_interface name="position"/>
-          <state_interface name="position"/>
-          <state_interface name="velocity"/>
-        </joint>
-      </xacro:if>
-      <!-- Only in fake hw mode (optional, but keep if you need it) -->
-      <xacro:if value="${use_fake_hardware}">
-        <gpio name="reactivate_gripper">
-          <command_interface name="reactivate_gripper_cmd"/>
-          <command_interface name="reactivate_gripper_response"/>
-        </gpio>
-      </xacro:if>
-    </ros2_control>
   </xacro:macro>
 </robot>
